File: esp32_midi/64buttons.kicad_sch (KiCad schematic)
At the start: 142 parts, among them SW11 SW_SPST, U17 BL1551, U18 BL1551, U19 BL1551, U20 BL1551, U21 BL1551, U22 BL1551, U23 BL1551, U24 BL1551, U25 BL1551, U26 BL1551, U27 BL1551, U28 BL1551, U29 BL1551, U30 BL1551, U31 BL1551

Commit message: Updated pcb
Parts:
- renumbered SW11 to SW10, SW11 to SW12, SW11 to SW13, SW11 to SW14, SW11 to SW15, SW11 to SW16, SW11 to SW17, SW11 to SW18, SW11 to SW19, SW11 to SW2, SW11 to SW20, SW11 to SW21, SW11 to SW22, SW11 to SW23, SW11 to SW24, SW11 to SW25, SW11 to SW26, SW11 to SW27, SW11 to SW28, SW11 to SW29, SW11 to SW3, SW11 to SW30, SW11 to SW31, SW11 to SW32, SW11 to SW33, SW11 to SW34, SW11 to SW35, SW11 to SW36, SW11 to SW37, SW11 to SW38, SW11 to SW39, SW11 to SW4, SW11 to SW40, SW11 to SW41, SW11 to SW42, SW11 to SW43, SW11 to SW44, SW11 to SW45, SW11 to SW46, SW11 to SW47, SW11 to SW48, SW11 to SW49, SW11 to SW5, SW11 to SW50, SW11 to SW51, SW11 to SW52, SW11 to SW53, SW11 to SW54, SW11 to SW55, SW11 to SW56, SW11 to SW57, SW11 to SW58, SW11 to SW59, SW11 to SW6, SW11 to SW60, SW11 to SW61, SW11 to SW62, SW11 to SW63, SW11 to SW64, SW11 to SW65, SW11 to SW7, SW11 to SW8, SW11 to SW9, U17 to U?, U31 to U?, U28 to U?, U22 to U?, U30 to U?, U24 to U?, U27 to U?, U20 to U?, U26 to U?, U18 to U?, U25 to U?, U21 to U?, U29 to U?, U19 to U?, U23 to U?
Connections:
- net SEL4: now reaches U?.6

Commit message: Add ordentliche-teile
Parts:
- SW10, SW11, SW12, SW13, SW14, SW15, SW16, SW17, SW18, SW19, SW2, SW20, SW21, SW22, SW23, SW24, SW25, SW26, SW27, SW28, SW29, SW3, SW30, SW31, SW32, SW33, SW34, SW35, SW36, SW37, SW38, SW39, SW4, SW40, SW41, SW42, SW43, SW44, SW45, SW46, SW47, SW48, SW49, SW5, SW50, SW51, SW52, SW53, SW54, SW55, SW56, SW57, SW58, SW59, SW6, SW60, SW61, SW62, SW63, SW64, SW65, SW7, SW8, SW9: footprint (none) -> ordentliche-teile:scheißbutton
