File: esp32_midi/analogorgie.kicad_sch (KiCad schematic)
At the start: 64 parts, among them U10 BL1551, U108 BL1551, U11 BL1551, U114 BL1551, U12 BL1551, U13 BL1551, U14 BL1551, U15 BL1551, U16 BL1551, U17 BL1551, U18 BL1551, U19 BL1551, U20 BL1551, U21 BL1551, U22 BL1551, U23 BL1551, U24 BL1551, U25 BL1551, U26 BL1551, U27 BL1551, U28 BL1551, U29 BL1551, U30 BL1551, U31 BL1551, U32 BL1551, U33 BL1551, U34 BL1551, U35 BL1551, U6 BL1551, U7 BL1551, U8 BL1551, U9 BL1551

Commit message: Started work on PCB
Connections:
- net OUTPUT renamed OUTPUT0
- no-connect marks 4 -> 3
Other:
- moved on the sheet: R?
Changed lines of the file:
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@@
 (kicad_sch (version 20230121) (generator eeschema)
-  (paper "A4")
+  (paper "A3")
   (junction (at 132.08 33.02) (diameter 0) (color 0 0 0 0)
   )
@@
   (no_connect (at 171.45 59.69))
   (no_connect (at 254 59.69))
-  (no_connect (at 335.28 59.69))
   (no_connect (at 90.17 59.69))
-  (wire (pts (xy 107.95 50.8) (xy 107.95 44.45))
+  (wire (pts (xy 107.95 50.8) (xy 107.95 45.72))
     (stroke (width 0) (type default))
   )
@@
     (stroke (width 0) (type default))
   )
-  (wire (pts (xy 271.78 50.8) (xy 271.78 44.45))
+  (wire (pts (xy 271.78 50.8) (xy 271.78 45.72))
     (stroke (width 0) (type default))
   )
@@
     (stroke (width 0) (type default))
   )
-  (wire (pts (xy 262.89 33.02) (xy 262.89 36.83))
+  (wire (pts (xy 262.89 33.02) (xy 262.89 38.1))
     (stroke (width 0) (type default))
   )
@@
     (stroke (width 0) (type default))
   )
-  (wire (pts (xy 99.06 50.8) (xy 99.06 44.45))
+  (wire (pts (xy 99.06 50.8) (xy 99.06 45.72))
     (stroke (width 0) (type default))
   )
@@
     (stroke (width 0) (type default))
   )
-  (wire (pts (xy 262.89 50.8) (xy 262.89 44.45))
+  (wire (pts (xy 262.89 50.8) (xy 262.89 45.72))
     (stroke (width 0) (type default))
   )
@@
     (stroke (width 0) (type default))
   )
-  (wire (pts (xy 266.7 40.64) (xy 266.7 46.99))
+  (wire (pts (xy 266.7 41.91) (xy 266.7 46.99))
     (stroke (width 0) (type default))
   )
@@
     (stroke (width 0) (type default))
   )
-  (wire (pts (xy 102.87 40.64) (xy 102.87 46.99))
+  (wire (pts (xy 102.87 41.91) (xy 102.87 46.99))
     (stroke (width 0) (type default))
   )
@@
     (stroke (width 0) (type default))
   )
-  (wire (pts (xy 107.95 33.02) (xy 107.95 36.83))
+  (wire (pts (xy 107.95 33.02) (xy 107.95 38.1))
     (stroke (width 0) (type default))
   )
@@
     (stroke (width 0) (type default))
   )
-  (wire (pts (xy 111.76 40.64) (xy 111.76 53.34))
+  (wire (pts (xy 111.76 41.91) (xy 111.76 53.34))
     (stroke (width 0) (type default))
   )
@@
     (stroke (width 0) (type default))
   )
-  (wire (pts (xy 99.06 33.02) (xy 99.06 36.83))
+  (wire (pts (xy 99.06 33.02) (xy 99.06 38.1))
     (stroke (width 0) (type default))
   )
@@
     (stroke (width 0) (type default))
   )
-  (wire (pts (xy 271.78 33.02) (xy 271.78 36.83))
+  (wire (pts (xy 271.78 33.02) (xy 271.78 38.1))
     (stroke (width 0) (type default))
   )
@@
     (stroke (width 0) (type default))
   )
-  (wire (pts (xy 275.59 40.64) (xy 275.59 53.34))
+  (wire (pts (xy 275.59 41.91) (xy 275.59 53.34))
     (stroke (width 0) (type default))
   )
@@
     (effects (font (size 1.27 1.27)) (justify left))
   )
-  (hierarchical_label "OUTPUT" (shape input) (at 170.18 129.54 0) (fields_autoplaced)
+  (hierarchical_label "OUTPUT0" (shape input) (at 170.18 129.54 0) (fields_autoplaced)
     (effects (font (size 1.27 1.27)) (justify left))
   )
@@
     )
   )
-  (symbol (lib_id "Device:R_Potentiometer") (at 271.78 40.64 0) (unit 1)
+  (symbol (lib_id "Device:R_Potentiometer") (at 271.78 41.91 0) (unit 1)
     (in_bom yes) (on_board yes) (dnp no)
-    (property "Reference" "R?" (at 278.13 39.37 0)
+    (property "Reference" "R?" (at 278.13 40.64 0)
       (effects (font (size 1.27 1.27)) (justify left))
     )
-    (property "Value" "R_Variable" (at 278.13 41.91 0)
+    (property "Value" "R_Variable" (at 278.13 43.18 0)
       (effects (font (size 1.27 1.27)) (justify left))
     )
-    (property "Footprint" "Potentiometer_THT:Potentiometer_Alps_RK09L_Single_Vertical" (at 271.78 40.64 0)
+    (property "Footprint" "Potentiometer_THT:Potentiometer_Alps_RK09L_Single_Vertical" (at 271.78 41.91 0)
       (effects (font (size 1.27 1.27)) hide)
     )
-    (property "Datasheet" "~" (at 271.78 40.64 0)
+    (property "Datasheet" "~" (at 271.78 41.91 0)
       (effects (font (size 1.27 1.27)) hide)
     )
@@
     )
   )
-  (symbol (lib_id "Device:R_Potentiometer") (at 262.89 40.64 0) (unit 1)
+  (symbol (lib_id "Device:R_Potentiometer") (at 262.89 41.91 0) (unit 1)
     (in_bom yes) (on_board yes) (dnp no)
-    (property "Reference" "R?" (at 269.24 39.37 0)
+    (property "Reference" "R?" (at 269.24 40.64 0)
       (effects (font (size 1.27 1.27)) (justify left))
     )
-    (property "Value" "R_Variable" (at 269.24 41.91 0)
+    (property "Value" "R_Variable" (at 269.24 43.18 0)
       (effects (font (size 1.27 1.27)) (justify left))
     )
-    (property "Footprint" "Potentiometer_THT:Potentiometer_Alps_RK09L_Single_Vertical" (at 262.89 40.64 0)
+    (property "Footprint" "Potentiometer_THT:Potentiometer_Alps_RK09L_Single_Vertical" (at 262.89 41.91 0)
       (effects (font (size 1.27 1.27)) hide)
     )
-    (property "Datasheet" "~" (at 262.89 40.64 0)
+    (property "Datasheet" "~" (at 262.89 41.91 0)
       (effects (font (size 1.27 1.27)) hide)
     )
@@
     )
   )
-  (symbol (lib_id "Device:R_Potentiometer") (at 99.06 40.64 0) (unit 1)
+  (symbol (lib_id "Device:R_Potentiometer") (at 99.06 41.91 0) (unit 1)
     (in_bom yes) (on_board yes) (dnp no)
-    (property "Reference" "R?" (at 105.41 39.37 0)
+    (property "Reference" "R?" (at 105.41 40.64 0)
       (effects (font (size 1.27 1.27)) (justify left))
     )
-    (property "Value" "R_Variable" (at 105.41 41.91 0)
+    (property "Value" "R_Variable" (at 105.41 43.18 0)
       (effects (font (size 1.27 1.27)) (justify left))
     )
-    (property "Footprint" "Potentiometer_THT:Potentiometer_Alps_RK09L_Single_Vertical" (at 99.06 40.64 0)
+    (property "Footprint" "Potentiometer_THT:Potentiometer_Alps_RK09L_Single_Vertical" (at 99.06 41.91 0)
       (effects (font (size 1.27 1.27)) hide)
     )
-    (property "Datasheet" "~" (at 99.06 40.64 0)
+    (property "Datasheet" "~" (at 99.06 41.91 0)
       (effects (font (size 1.27 1.27)) hide)
     )
@@
     )
   )
-  (symbol (lib_id "Device:R_Potentiometer") (at 107.95 40.64 0) (unit 1)
+  (symbol (lib_id "Device:R_Potentiometer") (at 107.95 41.91 0) (unit 1)
     (in_bom yes) (on_board yes) (dnp no)
-    (property "Reference" "R?" (at 114.3 39.37 0)
+    (property "Reference" "R?" (at 114.3 40.64 0)
       (effects (font (size 1.27 1.27)) (justify left))
     )
-    (property "Value" "R_Variable" (at 114.3 41.91 0)
+    (property "Value" "R_Variable" (at 114.3 43.18 0)
       (effects (font (size 1.27 1.27)) (justify left))
     )
-    (property "Footprint" "Potentiometer_THT:Potentiometer_Alps_RK09L_Single_Vertical" (at 107.95 40.64 0)
+    (property "Footprint" "Potentiometer_THT:Potentiometer_Alps_RK09L_Single_Vertical" (at 107.95 41.91 0)
       (effects (font (size 1.27 1.27)) hide)
     )
-    (property "Datasheet" "~" (at 107.95 40.64 0)
+    (property "Datasheet" "~" (at 107.95 41.91 0)
       (effects (font (size 1.27 1.27)) hide)
     )

Commit message: improve component spacing, add more LEDs
Parts:
- R? (x24): footprint Potentiometer_THT:Potentiometer_Alps_RK09L_Single_Vertical -> ordentliche-teile:Potentiometer_vom_markt
Changed lines of the file:
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@@
       (effects (font (size 1.27 1.27)) (justify left))
     )
-    (property "Footprint" "Potentiometer_THT:Potentiometer_Alps_RK09L_Single_Vertical" (at 271.78 41.91 0)
+    (property "Footprint" "ordentliche-teile:Potentiometer_vom_markt" (at 271.78 41.91 0)
       (effects (font (size 1.27 1.27)) hide)
     )
@@
       (effects (font (size 1.27 1.27)) (justify left))
     )
-    (property "Footprint" "Potentiometer_THT:Potentiometer_Alps_RK09L_Single_Vertical" (at 313.69 41.91 0)
+    (property "Footprint" "ordentliche-teile:Potentiometer_vom_markt" (at 313.69 41.91 0)
       (effects (font (size 1.27 1.27)) hide)
     )
@@
       (effects (font (size 1.27 1.27)) (justify left))
     )
-    (property "Footprint" "Potentiometer_THT:Potentiometer_Alps_RK09L_Single_Vertical" (at 187.96 41.91 0)
+    (property "Footprint" "ordentliche-teile:Potentiometer_vom_markt" (at 187.96 41.91 0)
       (effects (font (size 1.27 1.27)) hide)
     )
@@
       (effects (font (size 1.27 1.27)) (justify left))
     )
-    (property "Footprint" "Potentiometer_THT:Potentiometer_Alps_RK09L_Single_Vertical" (at 241.3 41.91 0)
+    (property "Footprint" "ordentliche-teile:Potentiometer_vom_markt" (at 241.3 41.91 0)
       (effects (font (size 1.27 1.27)) hide)
     )
@@
       (effects (font (size 1.27 1.27)) (justify left))
     )
-    (property "Footprint" "Potentiometer_THT:Potentiometer_Alps_RK09L_Single_Vertical" (at 123.19 41.91 0)
+    (property "Footprint" "ordentliche-teile:Potentiometer_vom_markt" (at 123.19 41.91 0)
       (effects (font (size 1.27 1.27)) hide)
     )
@@
       (effects (font (size 1.27 1.27)) (justify left))
     )
-    (property "Footprint" "Potentiometer_THT:Potentiometer_Alps_RK09L_Single_Vertical" (at 132.08 41.91 0)
+    (property "Footprint" "ordentliche-teile:Potentiometer_vom_markt" (at 132.08 41.91 0)
       (effects (font (size 1.27 1.27)) hide)
     )
@@
       (effects (font (size 1.27 1.27)) (justify left))
     )
-    (property "Footprint" "Potentiometer_THT:Potentiometer_Alps_RK09L_Single_Vertical" (at 287.02 41.91 0)
+    (property "Footprint" "ordentliche-teile:Potentiometer_vom_markt" (at 287.02 41.91 0)
       (effects (font (size 1.27 1.27)) hide)
     )
@@
       (effects (font (size 1.27 1.27)) (justify left))
     )
-    (property "Footprint" "Potentiometer_THT:Potentiometer_Alps_RK09L_Single_Vertical" (at 158.75 41.91 0)
+    (property "Footprint" "ordentliche-teile:Potentiometer_vom_markt" (at 158.75 41.91 0)
       (effects (font (size 1.27 1.27)) hide)
     )
@@
       (effects (font (size 1.27 1.27)) (justify left))
     )
-    (property "Footprint" "Potentiometer_THT:Potentiometer_Alps_RK09L_Single_Vertical" (at 322.58 41.91 0)
+    (property "Footprint" "ordentliche-teile:Potentiometer_vom_markt" (at 322.58 41.91 0)
       (effects (font (size 1.27 1.27)) hide)
     )
@@
       (effects (font (size 1.27 1.27)) (justify left))
     )
-    (property "Footprint" "Potentiometer_THT:Potentiometer_Alps_RK09L_Single_Vertical" (at 232.41 41.91 0)
+    (property "Footprint" "ordentliche-teile:Potentiometer_vom_markt" (at 232.41 41.91 0)
       (effects (font (size 1.27 1.27)) hide)
     )
@@
       (effects (font (size 1.27 1.27)) (justify left))
     )
-    (property "Footprint" "Potentiometer_THT:Potentiometer_Alps_RK09L_Single_Vertical" (at 114.3 41.91 0)
+    (property "Footprint" "ordentliche-teile:Potentiometer_vom_markt" (at 114.3 41.91 0)
       (effects (font (size 1.27 1.27)) hide)
     )
@@
       (effects (font (size 1.27 1.27)) (justify left))
     )
-    (property "Footprint" "Potentiometer_THT:Potentiometer_Alps_RK09L_Single_Vertical" (at 223.52 41.91 0)
+    (property "Footprint" "ordentliche-teile:Potentiometer_vom_markt" (at 223.52 41.91 0)
       (effects (font (size 1.27 1.27)) hide)
     )
@@
       (effects (font (size 1.27 1.27)) (justify left))
     )
-    (property "Footprint" "Potentiometer_THT:Potentiometer_Alps_RK09L_Single_Vertical" (at 262.89 41.91 0)
+    (property "Footprint" "ordentliche-teile:Potentiometer_vom_markt" (at 262.89 41.91 0)
       (effects (font (size 1.27 1.27)) hide)
     )
@@
       (effects (font (size 1.27 1.27)) (justify left))
     )
-    (property "Footprint" "Potentiometer_THT:Potentiometer_Alps_RK09L_Single_Vertical" (at 214.63 41.91 0)
+    (property "Footprint" "ordentliche-teile:Potentiometer_vom_markt" (at 214.63 41.91 0)
       (effects (font (size 1.27 1.27)) hide)
     )
@@
       (effects (font (size 1.27 1.27)) (justify left))
     )
-    (property "Footprint" "Potentiometer_THT:Potentiometer_Alps_RK09L_Single_Vertical" (at 278.13 41.91 0)
+    (property "Footprint" "ordentliche-teile:Potentiometer_vom_markt" (at 278.13 41.91 0)
       (effects (font (size 1.27 1.27)) hide)
     )
@@
       (effects (font (size 1.27 1.27)) (justify left))
     )
-    (property "Footprint" "Potentiometer_THT:Potentiometer_Alps_RK09L_Single_Vertical" (at 304.8 41.91 0)
+    (property "Footprint" "ordentliche-teile:Potentiometer_vom_markt" (at 304.8 41.91 0)
       (effects (font (size 1.27 1.27)) hide)
     )
@@
       (effects (font (size 1.27 1.27)) (justify left))
     )
-    (property "Footprint" "Potentiometer_THT:Potentiometer_Alps_RK09L_Single_Vertical" (at 196.85 41.91 0)
+    (property "Footprint" "ordentliche-teile:Potentiometer_vom_markt" (at 196.85 41.91 0)
       (effects (font (size 1.27 1.27)) hide)
     )
@@
       (effects (font (size 1.27 1.27)) (justify left))
     )
-    (property "Footprint" "Potentiometer_THT:Potentiometer_Alps_RK09L_Single_Vertical" (at 179.07 41.91 0)
+    (property "Footprint" "ordentliche-teile:Potentiometer_vom_markt" (at 179.07 41.91 0)
       (effects (font (size 1.27 1.27)) hide)
     )
@@
       (effects (font (size 1.27 1.27)) (justify left))
     )
-    (property "Footprint" "Potentiometer_THT:Potentiometer_Alps_RK09L_Single_Vertical" (at 149.86 41.91 0)
+    (property "Footprint" "ordentliche-teile:Potentiometer_vom_markt" (at 149.86 41.91 0)
       (effects (font (size 1.27 1.27)) hide)
     )
@@
       (effects (font (size 1.27 1.27)) (justify left))
     )
-    (property "Footprint" "Potentiometer_THT:Potentiometer_Alps_RK09L_Single_Vertical" (at 99.06 41.91 0)
+    (property "Footprint" "ordentliche-teile:Potentiometer_vom_markt" (at 99.06 41.91 0)
       (effects (font (size 1.27 1.27)) hide)
     )
@@
       (effects (font (size 1.27 1.27)) (justify left))
     )
-    (property "Footprint" "Potentiometer_THT:Potentiometer_Alps_RK09L_Single_Vertical" (at 107.95 41.91 0)
+    (property "Footprint" "ordentliche-teile:Potentiometer_vom_markt" (at 107.95 41.91 0)
       (effects (font (size 1.27 1.27)) hide)
     )
@@
       (effects (font (size 1.27 1.27)) (justify left))
     )
-    (property "Footprint" "Potentiometer_THT:Potentiometer_Alps_RK09L_Single_Vertical" (at 295.91 41.91 0)
+    (property "Footprint" "ordentliche-teile:Potentiometer_vom_markt" (at 295.91 41.91 0)
       (effects (font (size 1.27 1.27)) hide)
     )
@@
       (effects (font (size 1.27 1.27)) (justify left))
     )
-    (property "Footprint" "Potentiometer_THT:Potentiometer_Alps_RK09L_Single_Vertical" (at 205.74 41.91 0)
+    (property "Footprint" "ordentliche-teile:Potentiometer_vom_markt" (at 205.74 41.91 0)
       (effects (font (size 1.27 1.27)) hide)
     )
@@
       (effects (font (size 1.27 1.27)) (justify left))
     )
-    (property "Footprint" "Potentiometer_THT:Potentiometer_Alps_RK09L_Single_Vertical" (at 140.97 41.91 0)
-      (effects (font (size 1.27 1.27)) hide)
-    )
+    (property "Footprint" "ordentliche-teile:Potentiometer_vom_markt" (at 140.97 41.91 0)
+      (effects (font (size 1.27 1.27)) hide)
+    )
