File: esp32_midi/analogorgie.kicad_sch (KiCad schematic)
At the start: 64 parts, among them U10 BL1551, U108 BL1551, U11 BL1551, U114 BL1551, U12 BL1551, U13 BL1551, U14 BL1551, U15 BL1551, U16 BL1551, U17 BL1551, U18 BL1551, U19 BL1551, U20 BL1551, U21 BL1551, U22 BL1551, U23 BL1551, U24 BL1551, U25 BL1551, U26 BL1551, U27 BL1551, U28 BL1551, U29 BL1551, U30 BL1551, U31 BL1551, U32 BL1551, U33 BL1551, U34 BL1551, U35 BL1551, U6 BL1551, U7 BL1551, U8 BL1551, U9 BL1551

Commit message: muchos viasos
Parts:
- R? (x32): symbol Device:R_Potentiometer -> Device:R_Potentiometer_MountingPin
Connections:
- net GND: now also R?.2, R?.MP (MountPin), R?.MP (MountPin), R?.MP (MountPin), R?.MP (MountPin), R?.MP (MountPin), R?.MP (MountPin), R?.MP (MountPin), R?.MP (MountPin), R?.MP (MountPin), R?.MP (MountPin), R?.MP (MountPin), R?.MP (MountPin), R?.MP (MountPin), R?.MP (MountPin), R?.MP (MountPin), R?.MP (MountPin), R?.MP (MountPin), R?.MP (MountPin), R?.MP (MountPin), R?.MP (MountPin), R?.MP (MountPin), R?.MP (MountPin), R?.MP (MountPin), R?.MP (MountPin), R?.MP (MountPin), R?.MP (MountPin), R?.MP (MountPin), R?.MP (MountPin), R?.MP (MountPin), R?.MP (MountPin), R?.MP (MountPin), R?.MP (MountPin), U27.3
- no-connect marks 3 -> 1
Other:
- moved on the sheet: U108B, U10A, U10B, U114A, U11A, U11B, U12A, U12B, U13A, U13B, U14A, U14B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

Commit message: Everything changed
Parts:
- R? (x24): footprint ordentliche-teile:Potentiometer_vom_markt -> Potentiometer_THT:Potentiometer_Alps_RK09L_Single_Vertical

Commit message: First load of bug fixes
Parts:
- U10, U108, U11, U114, U12, U13, U14, U15, U16, U17, U18, U19, U20, U21, U22, U23, U24, U25, U26, U27, U28, U29, U30, U31, U32, U33, U34, U35, U6, U7, U8, U9: footprint Package_TO_SOT_SMD:SOT-363_SC-70-6 -> Package_SON:Fairchild_MicroPak-6_1.0x1.45mm_P0.5mm
Connections:
- net OUTPUT0 renamed OUTPUT

Commit message: Update parts numbers
Parts:
- R? (x32): Field-1 (none) -> ${DNP}
- U10, U108, U11, U114, U12, U13, U14, U15, U16, U17, U18, U19, U20, U21, U22, U23, U24, U25, U26, U27, U28, U29, U30, U31, U32, U33, U34, U35, U6, U7, U8, U9: footprint Package_SON:Fairchild_MicroPak-6_1.0x1.45mm_P0.5mm -> Package_TO_SOT_SMD:SOT-363_SC-70-6; Field-1 (none) -> ${DNP}
