File: esp32_midi/esp32_midi.kicad_pcb (KiCad board)
At the start: 2 copper layers, 172.5 x 392 mm, 440 parts, among them J1 Conn_Display, J2 5V-12V, J4 MIDI 1 OUT, J5 MIDI 1 IN, J6 MIDI 1 OUT, Q1 BSS138, Q2 SS8050_C2150, Q3 SS8050_C2150, Q4 BSS138, SW1 SW_SPST, SW10 SW_SPST, SW11 SW_SPST, SW12 SW_SPST, SW13 SW_SPST, SW14 SW_SPST, SW15 SW_SPST, SW16 SW_SPST, SW17 SW_SPST, SW18 SW_SPST, SW19 SW_SPST, SW2 SW_SPST, SW20 SW_SPST, SW21 SW_SPST, SW22 SW_SPST, SW23 SW_SPST, SW24 SW_SPST, SW25 SW_SPST, SW26 SW_SPST, SW27 SW_SPST, SW28 SW_SPST, SW29 SW_SPST, SW3 SW_SPST, SW30 SW_SPST, SW31 SW_SPST, SW32 SW_SPST, SW33 SW_SPST, SW34 SW_SPST, SW35 SW_SPST, SW36 SW_SPST, SW37 SW_SPST, SW38 SW_SPST, SW39 SW_SPST, SW4 SW_SPST, SW40 SW_SPST, SW41 SW_SPST, SW42 SW_SPST, SW43 SW_SPST, SW44 SW_SPST, SW45 SW_SPST, SW46 SW_SPST, SW47 SW_SPST, SW48 SW_SPST, SW49 SW_SPST, SW5 SW_SPST, SW50 SW_SPST, SW51 SW_SPST, SW52 SW_SPST, SW53 SW_SPST, SW54 SW_SPST, SW55 SW_SPST, SW56 SW_SPST, SW57 SW_SPST, SW58 SW_SPST, SW59 SW_SPST, SW6 SW_SPST, SW60 SW_SPST, SW61 SW_SPST, SW62 SW_SPST, SW63 SW_SPST, SW64 SW_SPST, SW65 SW_SPST, SW66 SW_SPST, SW67 SW_SPST, SW68 SW_SPST, SW69 SW_SPST, SW7 SW_SPST, SW70 SW_SPST, SW71 SW_SPST, SW72 SW_SPST, SW73 SW_SPST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

Commit message: More pcb routings
Parts:
- USB Midi: renamed from USBC2
- USB Serial: renamed from USBC1
- moved U66 5.70 mm to (189.7, 129.8)
- moved U98 5.35 mm to (239.1, 194.5)
- moved U75 5.31 mm to (189.6, 151.4)
- moved U93 4.99 mm to (324.7, 172.9)
- moved U123 4.94 mm to (325.1, 237.8)
- moved U82 4.90 mm to (296.6, 151.9)
- moved U120 4.81 mm to (281.9, 237.7)
- moved U59 4.80 mm to (232.4, 108.8)
- moved U61 4.78 mm to (275.8, 108.5)
- moved U49 4.75 mm to (232.5, 87.2)
- moved U85 4.74 mm to (189.7, 173.1)
- moved U83 4.70 mm to (324.9, 151.4)
- moved U46 4.69 mm to (189.4, 87.5)
- moved U71 4.67 mm to (276.1, 129.8)
- moved U118 4.67 mm to (238.8, 237.8)
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- renumbered D8 to 3.3V, D9 to 5V, D7 to RX, D6 to TX
Routing:
- net +3.3V: track 0.00 -> 3082.5 mm, vias 0 -> 39
- net +5V: track 0.00 -> 2206.7 mm, vias 0 -> 4
- net /analogorgie/SEL0: track 0.00 -> 2020.8 mm, vias 0 -> 42
- net /analogorgie/SEL1: track 0.00 -> 941.6 mm, vias 0 -> 15
- net +3V3: track 0.00 -> 730.4 mm, vias 0 -> 16
- net /analogorgie/SEL2: track 0.00 -> 421.8 mm, vias 0 -> 10
- net /analogorgie/SEL3: track 0.00 -> 409.2 mm, vias 0 -> 6
- net Net-(D228-DOUT): track 0.00 -> 347.2 mm, vias 0 -> 2
- net /analogorgie/SEL4: track 0.00 -> 338.4 mm, vias 0 -> 6
- net Net-(U104-Pad1): track 0.00 -> 276.1 mm, vias 0 -> 6
- net Net-(U119-Pad4): track 0.00 -> 213.5 mm, vias 0 -> 8
- net Net-(D116-DIN): track 0.00 -> 206.2 mm, vias 0 -> 4
- net Net-(D180-DIN): track 0.00 -> 199.5 mm, vias 0 -> 2
- net Net-(D196-DOUT): track 0.00 -> 190.2 mm, vias 0 -> 2
- net Net-(D164-DOUT): track 0.00 -> 188.0 mm, vias 0 -> 2
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