File: esp32_midi/dcdc_lm2596.kicad_sch (KiCad schematic)
At the start: 5 parts, among them U2 LM2596S-5

Commit message: Net improvements
Connections:
- net DICK0: now reaches D82.1 (K), L1.1, U2.2 (OUT)
- net OUT renamed DICK1
Changed lines of the file:
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@@
     (stroke (width 0) (type default))
+  )
+  (global_label "DICK0" (shape input) (at 66.04 30.48 90) (fields_autoplaced)
+    (effects (font (size 1.27 1.27)) (justify left))
+    (property "Intersheetrefs" "${INTERSHEET_REFS}" (at 66.04 21.9499 90)
+      (effects (font (size 1.27 1.27)) (justify left) hide)
+    )
+  )
+  (global_label "DICK1" (shape input) (at 73.66 30.48 0) (fields_autoplaced)
+    (effects (font (size 1.27 1.27)) (justify left))
+    (property "Intersheetrefs" "${INTERSHEET_REFS}" (at 82.1901 30.48 0)
+      (effects (font (size 1.27 1.27)) (justify left) hide)
+    )
   )
   (hierarchical_label "GND" (shape input) (at 40.64 17.78 0) (fields_autoplaced)

Commit message: Update parts numbers
Parts:
- C4, C5, D82, L1, U2: Field-1 (none) -> ${DNP}
Changed lines of the file:
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@@
+      (effects (font (size 1.27 1.27)) hide)
+    )
+    (property "Field-1" "${DNP}" (at 73.66 34.29 0)
+      (effects (font (size 1.27 1.27)) hide)
+    )
+    (property "Field-1" "${DNP}" (at 73.66 34.29 0)
       (effects (font (size 1.27 1.27)) hide)
     )
@@
       (effects (font (size 1.27 1.27)) hide)
     )
+    (property "Field-1" "${DNP}" (at 66.04 34.29 0)
+      (effects (font (size 1.27 1.27)) hide)
+    )
+    (property "Field-1" "${DNP}" (at 66.04 34.29 0)
+      (effects (font (size 1.27 1.27)) hide)
+    )
     (pin "1")
     (pin "2")
@@
     )
     (property "Description" "Inductor" (at 69.85 30.48 0)
+      (effects (font (size 1.27 1.27)) hide)
+    )
+    (property "Field-1" "${DNP}" (at 69.85 30.48 0)
+      (effects (font (size 1.27 1.27)) hide)
+    )
+    (property "Field-1" "${DNP}" (at 69.85 30.48 0)
       (effects (font (size 1.27 1.27)) hide)
     )
@@
       (effects (font (size 1.27 1.27)) hide)
     )
+    (property "Field-1" "${DNP}" (at 40.64 21.59 0)
+      (effects (font (size 1.27 1.27)) hide)
+    )
+    (property "Field-1" "${DNP}" (at 40.64 21.59 0)
+      (effects (font (size 1.27 1.27)) hide)
+    )
     (pin "1")
     (pin "2")
@@
       (effects (font (size 1.27 1.27)) hide)
     )
+    (property "Field-1" "${DNP}" (at 53.34 27.94 0)
+      (effects (font (size 1.27 1.27)) hide)
+    )
+    (property "Field-1" "${DNP}" (at 53.34 27.94 0)
+      (effects (font (size 1.27 1.27)) hide)
+    )
