File: esp32_midi/midi.kicad_sch (KiCad schematic)
At the start: 7 parts, among them J5 MIDI 1 IN, U4 4N25

Commit message: First load of bug fixes
Connections:
- no-connect marks 0 -> 3
Changed lines of the file:
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@@
   (junction (at 92.71 50.8) (diameter 0) (color 0 0 0 0)
   )
+  (no_connect (at 121.92 77.47))
+  (no_connect (at 137.16 77.47))
+  (no_connect (at 67.31 63.5))
   (wire (pts (xy 121.92 74.93) (xy 92.71 74.93))
     (stroke (width 0) (type default))
@@
       (effects (font (size 1.27 1.27)) hide)
     )
-    (property "Description" "" (at 92.71 66.04 0)
+    (property "Description" "Diode" (at 92.71 66.04 0)
+      (effects (font (size 1.27 1.27)) hide)
+    )
+    (property "Sim.Device" "D" (at 92.71 66.04 0)
+      (effects (font (size 1.27 1.27)) hide)
+    )
+    (property "Sim.Pins" "1=K 2=A" (at 92.71 66.04 0)
       (effects (font (size 1.27 1.27)) hide)
     )
@@
       (effects (font (size 1.27 1.27)) hide)
     )
-    (property "Description" "" (at 57.15 72.39 0)
+    (property "Description" "Resistor" (at 57.15 72.39 0)
       (effects (font (size 1.27 1.27)) hide)
     )
@@
       (effects (font (size 1.27 1.27)) (justify left) hide)
     )
-    (property "Description" "" (at 74.93 66.04 0)
+    (property "Description" "DC Optocoupler Base Connected, Vce 30V, CTR 20%, Viso 2500V, DIP6" (at 74.93 66.04 0)
       (effects (font (size 1.27 1.27)) hide)
     )
@@
       (effects (font (size 1.27 1.27)) hide)
     )
-    (property "Description" "" (at 64.77 80.01 0)
+    (property "Description" "Resistor" (at 64.77 80.01 0)
       (effects (font (size 1.27 1.27)) hide)
     )
@@
       (effects (font (size 1.27 1.27)) hide)
     )
-    (property "Description" "" (at 64.77 72.39 0)
+    (property "Description" "Light emitting diode" (at 64.77 72.39 0)
       (effects (font (size 1.27 1.27)) hide)
     )
@@
       (effects (font (size 1.27 1.27)) hide)
     )
-    (property "Description" "" (at 113.03 50.8 0)
+    (property "Description" "Resistor" (at 113.03 50.8 0)
       (effects (font (size 1.27 1.27)) hide)
     )
@@
       (effects (font (size 1.27 1.27)) hide)
     )
-    (property "Description" "" (at 129.54 77.47 0)
-      (effects (font (size 1.27 1.27)) hide)
-    )
+    (property "Description" "5-pin DIN connector (5-pin DIN-5 stereo)" (at 129.54 77.47 0)
+      (effects (font (size 1.27 1.27)) hide)
+    )

Commit message: Update parts numbers
Parts:
- D5, D6, J5, R11, R3, R4, U4: Field-1 (none) -> ${DNP}
Changed lines of the file:
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@@
+      (effects (font (size 1.27 1.27)) hide)
+    )
+    (property "Field-1" "${DNP}" (at 92.71 66.04 0)
+      (effects (font (size 1.27 1.27)) hide)
+    )
+    (property "Field-1" "${DNP}" (at 92.71 66.04 0)
       (effects (font (size 1.27 1.27)) hide)
     )
@@
     )
     (property "Description" "Resistor" (at 57.15 72.39 0)
+      (effects (font (size 1.27 1.27)) hide)
+    )
+    (property "Field-1" "${DNP}" (at 57.15 72.39 0)
+      (effects (font (size 1.27 1.27)) hide)
+    )
+    (property "Field-1" "${DNP}" (at 57.15 72.39 0)
       (effects (font (size 1.27 1.27)) hide)
     )
@@
     )
     (property "Description" "DC Optocoupler Base Connected, Vce 30V, CTR 20%, Viso 2500V, DIP6" (at 74.93 66.04 0)
+      (effects (font (size 1.27 1.27)) hide)
+    )
+    (property "Field-1" "${DNP}" (at 74.93 66.04 0)
+      (effects (font (size 1.27 1.27)) hide)
+    )
+    (property "Field-1" "${DNP}" (at 74.93 66.04 0)
       (effects (font (size 1.27 1.27)) hide)
     )
@@
       (effects (font (size 1.27 1.27)) hide)
     )
+    (property "Field-1" "${DNP}" (at 64.77 80.01 0)
+      (effects (font (size 1.27 1.27)) hide)
+    )
+    (property "Field-1" "${DNP}" (at 64.77 80.01 0)
+      (effects (font (size 1.27 1.27)) hide)
+    )
     (pin "1")
     (pin "2")
@@
       (effects (font (size 1.27 1.27)) hide)
     )
+    (property "Field-1" "${DNP}" (at 64.77 72.39 0)
+      (effects (font (size 1.27 1.27)) hide)
+    )
+    (property "Field-1" "${DNP}" (at 64.77 72.39 0)
+      (effects (font (size 1.27 1.27)) hide)
+    )
     (pin "1")
     (pin "2")
@@
       (effects (font (size 1.27 1.27)) hide)
     )
+    (property "Field-1" "${DNP}" (at 113.03 50.8 0)
+      (effects (font (size 1.27 1.27)) hide)
+    )
+    (property "Field-1" "${DNP}" (at 113.03 50.8 0)
+      (effects (font (size 1.27 1.27)) hide)
+    )
     (pin "1")
     (pin "2")
@@
       (effects (font (size 1.27 1.27)) hide)
     )
+    (property "Field-1" "${DNP}" (at 129.54 77.47 0)
+      (effects (font (size 1.27 1.27)) hide)
+    )
+    (property "Field-1" "${DNP}" (at 129.54 77.47 0)
+      (effects (font (size 1.27 1.27)) hide)
+    )
