File: esp32_midi/midi_in_thru_out.kicad_sch (KiCad schematic)
At the start: 0 parts

Commit message: Started work on PCB
Other:
- sheet MIDI OUT1 renamed MIDI OUT
Changed lines of the file:
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@@
     (stroke (width 0.1524) (type solid))
     (fill (color 0 0 0 0.0000))
-    (property "Sheetname" "MIDI OUT1" (at 129.54 74.2184 0)
+    (property "Sheetname" "MIDI OUT" (at 129.54 74.2184 0)
       (effects (font (size 1.27 1.27)) (justify left bottom))
     )

Commit message: Everything changed
Parts:
- added D6: LED, LED_SMD:LED_0603_1608Metric, symbol Device:LED
- added R11: 1k, Resistor_SMD:R_1206_3216Metric, symbol Device:R
Connections:
- net GND: now also R11.1
- net TX: now also D6.1 (K)
- new net: D6.2 (A), R11.2
Changed lines of the file:
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@@
-(kicad_sch (version 20230121) (generator eeschema)
+(kicad_sch (version 20230620) (generator eeschema)
   (paper "A4")
-  (wire (pts (xy 123.19 83.82) (xy 129.54 83.82))
+  (junction (at 118.11 86.36) (diameter 0) (color 0 0 0 0)
+  )
+  (wire (pts (xy 109.22 83.82) (xy 129.54 83.82))
     (stroke (width 0) (type default))
   )
@@
     (stroke (width 0) (type default))
   )
-  (wire (pts (xy 123.19 86.36) (xy 129.54 86.36))
+  (wire (pts (xy 109.22 86.36) (xy 118.11 86.36))
     (stroke (width 0) (type default))
   )
   (wire (pts (xy 123.19 88.9) (xy 129.54 88.9))
+    (stroke (width 0) (type default))
+  )
+  (wire (pts (xy 118.11 86.36) (xy 129.54 86.36))
     (stroke (width 0) (type default))
   )
@@
     (stroke (width 0) (type default))
   )
-  (label "TX" (at 123.19 86.36 0) (fields_autoplaced)
+  (label "TX" (at 109.22 86.36 0) (fields_autoplaced)
     (effects (font (size 1.27 1.27)) (justify left bottom))
   )
@@
     (effects (font (size 1.27 1.27)) (justify left bottom))
   )
-  (label "5V" (at 123.19 83.82 0) (fields_autoplaced)
+  (label "5V" (at 109.22 83.82 0) (fields_autoplaced)
     (effects (font (size 1.27 1.27)) (justify left bottom))
   )
@@
   )
   (hierarchical_label "TX" (shape input) (at 177.8 55.88 180) (fields_autoplaced)
+    (effects (font (size 1.27 1.27)) (justify right))
+  )
+  (hierarchical_label "GND" (shape input) (at 118.11 101.6 270) (fields_autoplaced)
     (effects (font (size 1.27 1.27)) (justify right))
   )
@@
     (effects (font (size 1.27 1.27)) (justify right))
   )
+  (symbol (lib_id "Device:LED") (at 118.11 90.17 270) (unit 1)
+    (in_bom yes) (on_board yes) (dnp no)
+    (property "Reference" "D6" (at 121.3166 92.3926 0)
+      (effects (font (size 1.27 1.27)) (justify right))
+    )
+    (property "Value" "LED" (at 119.5948 89.8882 0)
+      (effects (font (size 1.27 1.27)) (justify right))
+    )
+    (property "Footprint" "LED_SMD:LED_0603_1608Metric" (at 118.11 90.17 0)
+      (effects (font (size 1.27 1.27)) hide)
+    )
+    (property "Datasheet" "~" (at 118.11 90.17 0)
+      (effects (font (size 1.27 1.27)) hide)
+    )
+    (property "Description" "" (at 118.11 90.17 0)
+      (effects (font (size 1.27 1.27)) hide)
+    )
+    (property "LCSC Part #" "C2290" (at 118.11 90.17 0)
+      (effects (font (size 1.27 1.27)) hide)
+    )
+    (pin "1")
+    (pin "2")
+    (instances
+      (project "esp32_midi"
+        (path "/e33c0603-5c0d-4712-ab63-5756d1504b4c/2c215fe4-7c9a-4ae0-9a5d-913b04975b72"
+          (reference "D6") (unit 1)
+        )
+        (path "/e33c0603-5c0d-4712-ab63-5756d1504b4c/6690eb41-2c1d-4abf-90f8-fc4c3740650e/c474a483-652e-46b3-829f-20d9c40cc74b"
+          (reference "D237") (unit 1)
+        )
+        (path "/e33c0603-5c0d-4712-ab63-5756d1504b4c/6690eb41-2c1d-4abf-90f8-fc4c3740650e/067e608b-1500-4656-956d-29b5641ffb6f"
+          (reference "D238") (unit 1)
+        )
+        (path "/e33c0603-5c0d-4712-ab63-5756d1504b4c/6690eb41-2c1d-4abf-90f8-fc4c3740650e/23ac7157-3583-490b-a889-9bba9a4271ea"
+          (reference "D239") (unit 1)
+        )
+        (path "/e33c0603-5c0d-4712-ab63-5756d1504b4c/6690eb41-2c1d-4abf-90f8-fc4c3740650e"
+          (reference "D238") (unit 1)
+        )
+      )
+    )
+  )
+  (symbol (lib_id "Device:R") (at 118.11 97.79 180) (unit 1)
+    (in_bom yes) (on_board yes) (dnp no)
+    (property "Reference" "R11" (at 115.57 97.79 90)
+      (effects (font (size 1.27 1.27)) (justify left))
+    )
+    (property "Value" "1k" (at 115.57 95.25 90)
+      (effects (font (size 1.27 1.27)) (justify left))
+    )
+    (property "Footprint" "Resistor_SMD:R_1206_3216Metric" (at 119.888 97.79 90)
+      (effects (font (size 1.27 1.27)) hide)
+    )
+    (property "Datasheet" "~" (at 118.11 97.79 0)
+      (effects (font (size 1.27 1.27)) hide)
+    )
+    (property "Description" "" (at 118.11 97.79 0)
+      (effects (font (size 1.27 1.27)) hide)
+    )
+    (property "LCSC Part #" "C11702" (at 118.11 97.79 0)
+      (effects (font (size 1.27 1.27)) hide)
+    )
+    (pin "1")
+    (pin "2")
+    (instances
+      (project "esp32_midi"
+        (path "/e33c0603-5c0d-4712-ab63-5756d1504b4c/2c215fe4-7c9a-4ae0-9a5d-913b04975b72"
+          (reference "R11") (unit 1)
+        )
+        (path "/e33c0603-5c0d-4712-ab63-5756d1504b4c/6690eb41-2c1d-4abf-90f8-fc4c3740650e/c474a483-652e-46b3-829f-20d9c40cc74b"
+          (reference "R101") (unit 1)
+        )
+        (path "/e33c0603-5c0d-4712-ab63-5756d1504b4c/6690eb41-2c1d-4abf-90f8-fc4c3740650e/067e608b-1500-4656-956d-29b5641ffb6f"
+          (reference "R102") (unit 1)
+        )
+        (path "/e33c0603-5c0d-4712-ab63-5756d1504b4c/6690eb41-2c1d-4abf-90f8-fc4c3740650e/23ac7157-3583-490b-a889-9bba9a4271ea"
+          (reference "R103") (unit 1)
+        )
+        (path "/e33c0603-5c0d-4712-ab63-5756d1504b4c/6690eb41-2c1d-4abf-90f8-fc4c3740650e"
+          (reference "R102") (unit 1)
+        )
+      )
+    )
+  )
   (sheet (at 129.54 74.93) (size 15.24 17.78) (fields_autoplaced)

Commit message: First load of bug fixes
Changed lines of the file:
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@@
     (effects (font (size 1.27 1.27)) (justify left bottom))
+  )
+  (label "GND" (at 118.11 101.6 270) (fields_autoplaced)
+    (effects (font (size 1.27 1.27)) (justify right bottom))
   )
   (label "GND" (at 110.49 72.39 0) (fields_autoplaced)
@@
     (effects (font (size 1.27 1.27)) (justify right))
   )
-  (hierarchical_label "GND" (shape input) (at 118.11 101.6 270) (fields_autoplaced)
-    (effects (font (size 1.27 1.27)) (justify right))
-  )
   (hierarchical_label "3V3" (shape input) (at 177.8 50.8 180) (fields_autoplaced)
     (effects (font (size 1.27 1.27)) (justify right))
@@
       (effects (font (size 1.27 1.27)) hide)
     )
-    (property "Description" "" (at 118.11 90.17 0)
+    (property "Description" "Light emitting diode" (at 118.11 90.17 0)
       (effects (font (size 1.27 1.27)) hide)
     )
@@
       (effects (font (size 1.27 1.27)) hide)
     )
-    (property "Description" "" (at 118.11 97.79 0)
+    (property "Description" "Resistor" (at 118.11 97.79 0)
       (effects (font (size 1.27 1.27)) hide)
     )

Commit message: Update parts numbers
Parts:
- D6, R11: Field-1 (none) -> ${DNP}
Changed lines of the file:
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@@
+      (effects (font (size 1.27 1.27)) hide)
+    )
+    (property "Field-1" "${DNP}" (at 118.11 90.17 0)
+      (effects (font (size 1.27 1.27)) hide)
+    )
+    (property "Field-1" "${DNP}" (at 118.11 90.17 0)
       (effects (font (size 1.27 1.27)) hide)
     )
@@
       (effects (font (size 1.27 1.27)) hide)
     )
+    (property "Field-1" "${DNP}" (at 118.11 97.79 0)
+      (effects (font (size 1.27 1.27)) hide)
+    )
+    (property "Field-1" "${DNP}" (at 118.11 97.79 0)
+      (effects (font (size 1.27 1.27)) hide)
+    )
